File: The Open Bar.sch (KiCad schematic (older format))
At the start: 17 parts, among them P1 CONN_01X02, P2 CONN_01X02, P3 CONN_01X02, P4 CONN_01X02, P5 CONN_01X02, U1 AP3003-5.0V, U2 TC1262

Commit message: Rev B, Added Flywheel Diodes
Connections:
- no-connect marks 0 -> 4
Changed lines of the file:
@@
 Sheet 1 5
 Title "The Open Bar Control Board"
-Date "2016-08-04"
-Rev "A"
+Date "2017-02-25"
+Rev "B"
 Comp "The Open Bar"
 Comment1 ""
@@
 $EndComp
 $Comp
-L GND #PWR4
+L GND #PWR01
 U 1 1 56CF48E6
 P 1000 2050
-F 0 "#PWR4" H 1000 1800 50  0001 C CNN
+F 0 "#PWR01" H 1000 1800 50  0001 C CNN
 F 1 "GND" H 1000 1900 50  0000 C CNN
 F 2 "" H 1000 2050 50  0000 C CNN
@@
 $EndComp
 $Comp
-L +3.3V #PWR2
+L +3.3V #PWR02
 U 1 1 56CF48E7
 P 800 950
-F 0 "#PWR2" H 800 800 50  0001 C CNN
+F 0 "#PWR02" H 800 800 50  0001 C CNN
 F 1 "+3.3V" H 800 1090 50  0000 C CNN
 F 2 "" H 800 950 50  0000 C CNN
@@
 $EndComp
 $Comp
-L +5V #PWR3
+L +5V #PWR03
 U 1 1 56CF48E8
 P 1000 1800
-F 0 "#PWR3" H 1000 1650 50  0001 C CNN
+F 0 "#PWR03" H 1000 1650 50  0001 C CNN
 F 1 "+5V" H 1000 1940 50  0000 C CNN
 F 2 "" H 1000 1800 50  0000 C CNN
@@
 $EndComp
 $Comp
-L GND #PWR1
+L GND #PWR04
 U 1 1 56CF48E9
 P 750 1100
-F 0 "#PWR1" H 750 850 50  0001 C CNN
+F 0 "#PWR04" H 750 850 50  0001 C CNN
 F 1 "GND" H 750 950 50  0000 C CNN
 F 2 "" H 750 1100 50  0000 C CNN
@@
 $EndSheet
 $Comp
-L +3.3V #PWR17
+L +3.3V #PWR05
 U 1 1 56D7C8D0
 P 7500 750
-F 0 "#PWR17" H 7500 600 50  0001 C CNN
+F 0 "#PWR05" H 7500 600 50  0001 C CNN
 F 1 "+3.3V" H 7500 890 50  0000 C CNN
 F 2 "" H 7500 750 50  0000 C CNN
@@
 Connection ~ 7950 4350
 $Comp
-L GND #PWR18
+L GND #PWR06
 U 1 1 56D80EBC
 P 7650 2100
-F 0 "#PWR18" H 7650 1850 50  0001 C CNN
+F 0 "#PWR06" H 7650 1850 50  0001 C CNN
 F 1 "GND" H 7650 1950 50  0000 C CNN
 F 2 "" H 7650 2100 50  0000 C CNN
@@
 $EndComp
 $Comp
-L +3.3V #PWR23
+L +3.3V #PWR07
 U 1 1 56D819AD
 P 7800 3500
-F 0 "#PWR23" H 7800 3350 50  0001 C CNN
+F 0 "#PWR07" H 7800 3350 50  0001 C CNN
 F 1 "+3.3V" H 7800 3640 50  0000 C CNN
 F 2 "" H 7800 3500 50  0000 C CNN
@@
 $EndComp
 $Comp
-L GND #PWR19
+L GND #PWR08
 U 1 1 56D819B3
 P 7650 3400
-F 0 "#PWR19" H 7650 3150 50  0001 C CNN
+F 0 "#PWR08" H 7650 3150 50  0001 C CNN
 F 1 "GND" H 7650 3250 50  0000 C CNN
 F 2 "" H 7650 3400 50  0000 C CNN
@@
 $EndComp
 $Comp
-L +3.3V #PWR20
+L +3.3V #PWR09
 U 1 1 56D81A6D
 P 7650 4500
-F 0 "#PWR20" H 7650 4350 50  0001 C CNN
+F 0 "#PWR09" H 7650 4350 50  0001 C CNN
 F 1 "+3.3V" H 7650 4640 50  0000 C CNN
 F 2 "" H 7650 4500 50  0000 C CNN
@@
 $EndComp
 $Comp
-L GND #PWR21
+L GND #PWR010
 U 1 1 56D81A73
 P 7650 4700
-F 0 "#PWR21" H 7650 4450 50  0001 C CNN
+F 0 "#PWR010" H 7650 4450 50  0001 C CNN
 F 1 "GND" H 7650 4550 50  0000 C CNN
 F 2 "" H 7650 4700 50  0000 C CNN
@@
 $EndComp
 $Comp
-L +3.3V #PWR22
+L +3.3V #PWR011
 U 1 1 56D81B2D
 P 7650 5750
-F 0 "#PWR22" H 7650 5600 50  0001 C CNN
+F 0 "#PWR011" H 7650 5600 50  0001 C CNN
 F 1 "+3.3V" H 7650 5890 50  0000 C CNN
 F 2 "" H 7650 5750 50  0000 C CNN
@@
 $EndComp
 $Comp
-L GND #PWR6
+L GND #PWR012
 U 1 1 56D9FCBF
 P 1650 1150
-F 0 "#PWR6" H 1650 900 50  0001 C CNN
+F 0 "#PWR012" H 1650 900 50  0001 C CNN
 F 1 "GND" H 1650 1000 50  0000 C CNN
 F 2 "" H 1650 1150 50  0000 C CNN
@@
 $EndComp
 $Comp
-L +12V #PWR8
+L +12V #PWR013
 U 1 1 56DA0F30
 P 1800 1950
-F 0 "#PWR8" H 1800 1800 50  0001 C CNN
+F 0 "#PWR013" H 1800 1800 50  0001 C CNN
 F 1 "+12V" H 1800 2090 50  0000 C CNN
 F 2 "" H 1800 1950 50  0000 C CNN
@@
 $EndComp
 $Comp
-L +12VA #PWR7
+L +12VA #PWR014
 U 1 1 56DA11C1
 P 1650 2200
-F 0 "#PWR7" H 1650 2050 50  0001 C CNN
+F 0 "#PWR014" H 1650 2050 50  0001 C CNN
 F 1 "+12VA" H 1650 2340 50  0000 C CNN
 F 2 "" H 1650 2200 50  0000 C CNN
@@
 	1650 2250 1650 2200
 $Comp
-L +12VA #PWR5
+L +12VA #PWR015
 U 1 1 56DA4A10
 P 1650 850
-F 0 "#PWR5" H 1650 700 50  0001 C CNN
+F 0 "#PWR015" H 1650 700 50  0001 C CNN
 F 1 "+12VA" H 1650 990 50  0000 C CNN
 F 2 "" H 1650 850 50  0000 C CNN
@@
 $EndComp
 $Comp
-L GND #PWR11
+L GND #PWR016
 U 1 1 56DAA647
 P 3650 3850
-F 0 "#PWR11" H 3650 3600 50  0001 C CNN
+F 0 "#PWR016" H 3650 3600 50  0001 C CNN
 F 1 "GND" H 3650 3700 50  0000 C CNN
 F 2 "" H 3650 3850 50  0000 C CNN
@@
 $EndComp
 $Comp
-L +12VA #PWR9
+L +12VA #PWR017
 U 1 1 56DAF69E
 P 2550 3350
-F 0 "#PWR9" H 2550 3200 50  0001 C CNN
+F 0 "#PWR017" H 2550 3200 50  0001 C CNN
 F 1 "+12VA" H 2550 3490 50  0000 C CNN
 F 2 "" H 2550 3350 50  0000 C CNN
@@
 Connection ~ 5150 3350
 $Comp
-L +5V #PWR14
+L +5V #PWR018
 U 1 1 56DB7AED
 P 5550 3350
-F 0 "#PWR14" H 5550 3200 50  0001 C CNN
+F 0 "#PWR018" H 5550 3200 50  0001 C CNN
 F 1 "+5V" H 5550 3490 50  0000 C CNN
 F 2 "" H 5550 3350 50  0000 C CNN
@@
 $EndComp
 $Comp
-L GND #PWR12
+L GND #PWR019
 U 1 1 56DC249F
 P 3750 5650
-F 0 "#PWR12" H 3750 5400 50  0001 C CNN
+F 0 "#PWR019" H 3750 5400 50  0001 C CNN
 F 1 "GND" H 3750 5500 50  0000 C CNN
 F 2 "" H 3750 5650 50  0000 C CNN
@@
 	4150 5150 4600 5150
 $Comp
-L +3.3V #PWR13
+L +3.3V #PWR020
 U 1 1 56DC4CA1
 P 4600 5150
-F 0 "#PWR13" H 4600 5000 50  0001 C CNN
+F 0 "#PWR020" H 4600 5000 50  0001 C CNN
 F 1 "+3.3V" H 4600 5290 50  0000 C CNN
 F 2 "" H 4600 5150 50  0000 C CNN
@@
 Connection ~ 4300 5150
 $Comp
-L +5V #PWR10
+L +5V #PWR021
 U 1 1 56DC6453
 P 2700 5150
-F 0 "#PWR10" H 2700 5000 50  0001 C CNN
+F 0 "#PWR021" H 2700 5000 50  0001 C CNN
 F 1 "+5V" H 2700 5290 50  0000 C CNN
 F 2 "" H 2700 5150 50  0000 C CNN
@@
 $EndComp
 $Comp
-L GND #PWR16
+L GND #PWR022
 U 1 1 57A4830D
 P 6950 2600
-F 0 "#PWR16" H 6950 2350 50  0001 C CNN
+F 0 "#PWR022" H 6950 2350 50  0001 C CNN
 F 1 "GND" H 6950 2450 50  0000 C CNN
 F 2 "" H 6950 2600 50  0000 C CNN
@@
 $EndComp
 $Comp
-L +3.3V #PWR15
+L +3.3V #PWR023
 U 1 1 57A48FC9
 P 6950 1650
-F 0 "#PWR15" H 6950 1500 50  0001 C CNN
+F 0 "#PWR023" H 6950 1500 50  0001 C CNN
 F 1 "+3.3V" H 6950 1790 50  0000 C CNN
 F 2 "" H 6950 1650 50  0000 C CNN
@@
 Text Notes 2350 6050 0    50   ~ 10
 If Making an addon board. Do not populate regulators.\nJumper the 3.3V, I2C, and Switch Connectors, de-populate R2, and populate R1.
+NoConn ~ 8550 2150
+NoConn ~ 8550 3500
+NoConn ~ 8550 4750
+NoConn ~ 8550 6000
 $EndSCHEMATC
